Commit message: parameters updated (length) some minor issues

File: description/robot_core.xacro (robot description, xacro)
@@ -1,18 +1,21 @@
 <?xml version="1.0"?>
-<robot xmlns:xacro="http://www.ros.org/wiki/xacro">
+<robot xmlns:xacro="http://www.ros.org/wiki/xacro" >
     <xacro:include filename="inertial_macros.xacro"/>
+   <xacro:property name="chassis_width" value="0.4"/>
+    <xacro:property name="chassis_height" value="0.08"/>
+    <xacro:property name="chassis_mass" value="6.0"/>
+    <xacro:property name="wheel_mass" value="2.1"/>
+    <xacro:property name="caster_wheel_mass" value="2.5"/>
+    <xacro:property name="caster_wheel_radius" value="0.0405"/>
+    <xacro:property name="wheel_thickness" value="0.045"/>
+    <xacro:property name="wheel_offset_z" value="0.01"/>
     <xacro:property name="chassis_length" value="0.5"/>
-    <xacro:property name="chassis_width" value="0.4"/>
-    <xacro:property name="chassis_height" value="0.1"/>
-    <xacro:property name="chassis_mass" value="6.0"/>
-    <xacro:property name="wheel_radius" value="0.081"/>
-    <xacro:property name="wheel_thickness" value="0.045"/>
-    <xacro:property name="wheel_mass" value="2.1"/>
-    <xacro:property name="wheel_offset_x" value="0.2"/>
-    <xacro:property name="wheel_offset_y" value="0.225"/>
-    <xacro:property name="wheel_offset_z" value="0.01"/>
-    <xacro:property name="caster_wheel_radius" value="0.0405"/>
-    <xacro:property name="caster_wheel_mass" value="2.5"/>
-    <xacro:property name="caster_wheel_offset_x" value="0.05"/>
+    <xacro:property name="wheel_offset_x" value="0.3373"/><!-- minor  change   -->
+    <xacro:property name="wheel_radius" value="0.033"/>  <!-- dont change   -->
+    <xacro:property name="wheel_offset_y" value="0.1485"/> <!-- dont change   -->
+    <!-- <xacro:property name="wheel_radius" value="0.033"/>     -->
+    <!-- <xacro:property name="wheel_offset_x" value="0.3373"/> -->
+    <!-- <xacro:property name="wheel_offset_y" value="0.1485"/>     -->
+    <xacro:property name="caster_wheel_offset_x" value="0.075"/>
     <xacro:property name="caster_wheel_offset_z" value="${wheel_offset_z - wheel_radius + caster_wheel_radius}"/>
     <material name="white">
@@ -62,5 +65,5 @@
             </geometry>
         </collision>
-        <xacro:inertial_box mass="6.0" x="${chassis_length}" y="${chassis_width}" z="${chassis_height}">
+        <xacro:inertial_box mass="0.5" x="${chassis_length}" y="${chassis_width}" z="${chassis_height}">
             <origin xyz="${chassis_length/2} 0 ${chassis_height/2}" rpy="0 0 0"/>
         </xacro:inertial_box>
@@ -73,5 +76,5 @@
         <parent link="base_link"/>
         <child link="left_wheel"/>
-        <origin xyz="${wheel_offset_x} ${wheel_offset_y} 0" rpy="-${pi/2} 0 0" />
+        <origin xyz="0 ${wheel_offset_y} 0" rpy="-${pi/2} 0 0" />
         <axis xyz="0 0 1"/>
     </joint>
@@ -99,5 +102,5 @@
         <parent link="base_link"/>
         <child link="right_wheel"/>
-        <origin xyz="${wheel_offset_x} ${-wheel_offset_y} 0" rpy="${pi/2} 0 0" />
+        <origin xyz="0 ${-wheel_offset_y} 0" rpy="${pi/2} 0 0" />
         <axis xyz="0 0 -1"/>
     </joint>
